File: cy8ckit-059_grbl_board.sch (KiCad schematic (older format))
At the start: 24 parts, among them IC1 CY8CKIT-059, J1 Connector:Conn_01x04_Male, J10 Conn_02x01, J11 Conn_02x01, J12 Conn_02x04_Odd_Even, J13 Conn_02x03_Odd_Even, J2 Connector:Conn_01x04_Male, J3 Connector:Conn_01x04_Male, J4 Conn_02x03_Odd_Even, J5 Conn_02x03_Odd_Even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

Commit message: V2.0
Parts:
- removed J13: Conn_02x03_Odd_Even, Socket_Strips:Socket_Strip_Straight_2x03_Pitch2.54mm, symbol Connector_Generic:Conn_02x03_Odd_Even
- removed J8: Conn_02x05_Odd_Even, Socket_Strips:Socket_Strip_Straight_2x05_Pitch2.54mm, symbol Connector_Generic:Conn_02x05_Odd_Even
- added C4, C5, C6: 100nF, Capacitors_THT:C_Disc_D3.8mm_W2.6mm_P2.50mm, symbol Device:C
- added J14: Conn_02x06_Odd_Even, Socket_Strips:Socket_Strip_Straight_2x06_Pitch2.54mm, symbol Connector_Generic:Conn_02x06_Odd_Even
- added J15: Conn_01x02_Male, Socket_Strips:Socket_Strip_Straight_1x02_Pitch2.54mm, symbol Connector:Conn_01x02_Male
- added J7: Conn_01x04_Male, Socket_Strips:Socket_Strip_Straight_1x04_Pitch2.54mm, symbol Connector:Conn_01x04_Male
- added R1, R2: R, Resistors_THT:R_Axial_DIN0207_L6.3mm_D2.5mm_P7.62mm_Horizontal, symbol Device:R
- J10: renamed from J9; footprint Sockets_MOLEX_KK-System:Socket_MOLEX-KK-RM2-54mm_Lock_2pin_straight -> Connectors_Terminal_Blocks:TerminalBlock_bornier-2_P5.08mm
- renumbered J10 to J11, J11 to J12, J12 to J13, J7 to J9
Connections:
- net +36V: now also R1.1
- net +5V: now also J15.1 (Pin_1), J7.3 (Pin_3); no longer A1.13 (~RST), A1.14 (~SLP), A2.13 (~RST), A2.14 (~SLP), A3.13 (~RST), A3.14 (~SLP)
- net GND: now also IC1.48 (P0_6), R2.2
- net GNDD: now also C4.2, C5.2, C6.2, J14.10 (Pin_10), J14.12 (Pin_12), J14.2 (Pin_2), J14.4 (Pin_4), J14.6 (Pin_6), J14.8 (Pin_8), J15.2 (Pin_2), J7.4 (Pin_4)
- net dir_x: now also IC1.43 (P0_1); no longer IC1.47 (P0_5)
- net dir_z: now also IC1.29 (P3_1); no longer IC1.28 (P3_0)
- net limit_x: now also C4.1, J14.1 (Pin_1), J14.3 (Pin_3)
- net limit_y: now also C5.1, J14.5 (Pin_5), J14.7 (Pin_7)
- net limit_z: now also C6.1, J14.11 (Pin_11), J14.9 (Pin_9)
- net step_x: now also IC1.44 (SAR1/P0_2); no longer IC1.48 (P0_6)
- net step_z: now also IC1.30 (EXT_REF1/P3_2); no longer IC1.29 (P3_1)
- net uart_rx: now reaches IC1.10 (P12_6/UART_RX)
- net uart_rx: now also J7.1 (Pin_1)
- net sleep_z: now reaches IC1.31 (P3_3)
- net sleep_z: now also A3.14 (~SLP)
- net reset_z: now reaches IC1.32 (P3_4)
- net reset_z: now also A3.13 (~RST)
- net enable_z: now reaches IC1.33 (P3_5)
- net enable_z: now also A3.9 (~EN)
- net fault_y: now reaches IC1.36 (P15_0)
- net fault_y: now also A2.2 (~FLT)
- net reset_y: now reaches IC1.40 (CMOD/P15_4)
- net reset_y: now also A2.13 (~RST)
- net enable_y: now reaches IC1.41 (P15_5)
- net enable_y: now also A2.9 (~EN)
- net fault_x: now reaches IC1.42 (P0_0)
- net fault_x: now also A1.2 (~FLT)
- net sleep_x: now reaches IC1.45 (EXT_REF0/P0_3)
- net sleep_x: now also A1.14 (~SLP)
- net reset_x: now reaches IC1.46 (SAR0/P0_4)
- net reset_x: now also A1.13 (~RST)
- net uart_tx: now reaches IC1.9 (P12_7/UART_TX)
- net uart_tx: now also J7.2 (Pin_2)
- net fault_z: now reaches A3.2 (~FLT)
- net fault_z: now also IC1.28 (P3_0)
- net step_enable_x renamed enable_x
- net enable_x: now also IC1.47 (P0_5); no longer IC1.49 (P0_7)
- net step_enable_y renamed sleep_y
- net sleep_y: now also A2.14 (~SLP); no longer A2.9 (~EN)
- removed net step_enable_z: A3.9 (~EN), IC1.30 (EXT_REF1/P3_2)
- new net motor_voltage: IC1.49 (P0_7), R1.2, R2.1
Other:
- moved on the sheet: J11, J12, J13, J9
